File: EbikeSupeMon.sch (KiCad schematic (older format))
At the start: 14 parts

Commit message: push before branch
Parts:
- C1, C2: renamed from C?; footprint (none) -> Capacitor_SMD:C_0805_2012Metric
- J1: renamed from J?; footprint (none) -> Connector_USB:USB_Micro-B_Wuerth_629105150521
- J2, J3: renamed from J?; footprint (none) -> Connector_PinHeader_2.54mm:PinHeader_1x02_P2.54mm_Horizontal
- R1, R2, R3, R4: renamed from R?; footprint (none) -> Resistor_SMD:R_0805_2012Metric
- SW1, SW2: renamed from SW?; footprint (none) -> Button_Switch_SMD:SW_SPST_B3U-1000P-B
- SW3: renamed from SW?; footprint (none) -> Button_Switch_SMD:SW_SPST_EVQPE1
- U1: renamed from U?; footprint (none) -> Package_DFN_QFN:TQFN-28-1EP_5x5mm_P0.5mm_EP3.25x3.25mm_ThermalVias
- gave numbers to parts that had none: 1
Connections:
- net BarrVRead renamed BattVRead
- no-connect marks 18 -> 46
