File: EbikeSupeMon.sch (KiCad schematic (older format))
At the start: 14 parts, among them J1 USB_B_Micro, J2 Key switch, J3 Controller enable, SW1 IO_0, SW2 EN, SW3 USB-Reg_EN, U1 CP2102N-QFN28, U2 ESP32-WROOM-32

Commit message: Time for layout!
Parts:
- C1: value 4.7uF -> 4.7uF X5R
- C2: value 0.1uF -> 0.1uF X5R
Connections:
- net 12V_I_mon: now reaches U2.9 (IO33)
- no-connect marks 46 -> 45
Changed lines of the file:
@@
 F7 "3.3Reg" O R 1450 7550 50
 F8 "5v_Bus" I R 1450 6600 50
+F9 "12V_I_mon" I L 750 6650 50
 $EndSheet
 $Comp
@@
 P 1350 2150
 F 0 "C1" H 1465 2196 50  0000 L CNN
-F 1 "4.7uF" H 1465 2105 50  0000 L CNN
+F 1 "4.7uF X5R" H 1465 2105 50  0000 L CNN
 F 2 "Capacitor_SMD:C_0805_2012Metric" H 1388 2000 50  0001 C CNN
 F 3 "~" H 1350 2150 50  0001 C CNN
@@
 P 1700 2150
 F 0 "C2" H 1815 2196 50  0000 L CNN
-F 1 "0.1uF" H 1815 2105 50  0000 L CNN
+F 1 "0.1uF X5R" H 1815 2105 50  0000 L CNN
 F 2 "Capacitor_SMD:C_0805_2012Metric" H 1738 2000 50  0001 C CNN
 F 3 "~" H 1700 2150 50  0001 C CNN
@@
 NoConn ~ 9800 4100
 NoConn ~ 9800 4200
-NoConn ~ 9800 4300
 NoConn ~ 8600 3900
 NoConn ~ 8600 3800
@@
 NoConn ~ 8600 2500
 NoConn ~ 1450 6900
+Text Label 650  6550 1    50   ~ 0
+12V_I_mon
+Wire Wire Line
+	650  6550 650  6650
+Wire Wire Line
+	650  6650 750  6650
+Text Label 10000 4300 0    50   ~ 0
+12V_I_mon
+Wire Wire Line
+	10000 4300 9800 4300
 $EndSCHEMATC
