File: _autosave-EbikeSupeMon.sch (KiCad schematic (older format))
At the start: 15 parts, among them J1 USB_B_Micro, J2 Key switch, J3 Controller enable, SW1 IO_0, SW2 EN, SW3 USB-Reg_EN, U1 CP2102N-QFN28, U2 ESP32-WROOM-32

Commit message: rev 2 done
Parts:
- J6: renamed from J?; footprint (none) -> Connector_USB:USB_A_CONNFLY_DS1095-WNR0
Changed lines of the file:
@@
 	10000 4300 9800 4300
 $Comp
-L Connector:USB_A J?
+L Connector:USB_A J6
 U 1 1 5F6904F4
 P 5700 1150
-F 0 "J?" H 5757 1617 50  0000 C CNN
+F 0 "J6" H 5757 1617 50  0000 C CNN
 F 1 "USB_A" H 5757 1526 50  0000 C CNN
-F 2 "" H 5850 1100 50  0001 C CNN
+F 2 "Connector_USB:USB_A_CONNFLY_DS1095-WNR0" H 5850 1100 50  0001 C CNN
 F 3 " ~" H 5850 1100 50  0001 C CNN
 	1    5700 1150
@@
 $EndComp
 $Comp
-L power:+5V #PWR?
+L power:+5V #PWR0143
 U 1 1 5F694187
 P 6150 950
-F 0 "#PWR?" H 6150 800 50  0001 C CNN
+F 0 "#PWR0143" H 6150 800 50  0001 C CNN
 F 1 "+5V" V 6165 1078 50  0000 L CNN
 F 2 "" H 6150 950 50  0001 C CNN
@@
 NoConn ~ 6000 1250
 $Comp
-L power:GND #PWR?
+L power:GND #PWR0144
 U 1 1 5F696EE2
 P 5650 1650
-F 0 "#PWR?" H 5650 1400 50  0001 C CNN
+F 0 "#PWR0144" H 5650 1400 50  0001 C CNN
 F 1 "GND" H 5655 1477 50  0000 C CNN
 F 2 "" H 5650 1650 50  0001 C CNN
